File: postcard/postcard.sch (KiCad schematic (older format))
At the start: 20 parts, among them SW1 SW_Push, U1 ATtiny85-20SU

Commit message: tsv added
Parts:
- R1: value R -> 10k
- R2, R3, R4, R5: value R -> 100
- U1: symbol MCU_Microchip_ATtiny:ATtiny85-20SU -> postcard-rescue:ATtiny85-20SU-MCU_Microchip_ATtiny
Changed lines of the file:
@@
 P 3250 1500
 F 0 "R2" V 3043 1500 50  0000 C CNN
-F 1 "R" V 3134 1500 50  0000 C CNN
+F 1 "100" V 3134 1500 50  0000 C CNN
 F 2 "Resistor_SMD:R_0805_2012Metric_Pad1.15x1.40mm_HandSolder" V 3180 1500 50  0001 C CNN
 F 3 "~" H 3250 1500 50  0001 C CNN
@@
 P 3250 2000
 F 0 "R3" V 3043 2000 50  0000 C CNN
-F 1 "R" V 3134 2000 50  0000 C CNN
+F 1 "100" V 3134 2000 50  0000 C CNN
 F 2 "Resistor_SMD:R_0805_2012Metric_Pad1.15x1.40mm_HandSolder" V 3180 2000 50  0001 C CNN
 F 3 "~" H 3250 2000 50  0001 C CNN
@@
 P 3250 2500
 F 0 "R4" V 3043 2500 50  0000 C CNN
-F 1 "R" V 3134 2500 50  0000 C CNN
+F 1 "100" V 3134 2500 50  0000 C CNN
 F 2 "Resistor_SMD:R_0805_2012Metric_Pad1.15x1.40mm_HandSolder" V 3180 2500 50  0001 C CNN
 F 3 "~" H 3250 2500 50  0001 C CNN
@@
 P 3300 3050
 F 0 "R5" V 3093 3050 50  0000 C CNN
-F 1 "R" V 3184 3050 50  0000 C CNN
+F 1 "100" V 3184 3050 50  0000 C CNN
 F 2 "Resistor_SMD:R_0805_2012Metric_Pad1.15x1.40mm_HandSolder" V 3230 3050 50  0001 C CNN
 F 3 "~" H 3300 3050 50  0001 C CNN
@@
 P 2500 3100
 F 0 "R1" V 2293 3100 50  0000 C CNN
-F 1 "R" V 2384 3100 50  0000 C CNN
+F 1 "10k" V 2384 3100 50  0000 C CNN
 F 2 "Resistor_SMD:R_0805_2012Metric_Pad1.15x1.40mm_HandSolder" V 2430 3100 50  0001 C CNN
 F 3 "~" H 2500 3100 50  0001 C CNN
@@
 	2200 1500 2200 1650
 $Comp
-L MCU_Microchip_ATtiny:ATtiny85-20SU U1
+L postcard-rescue:ATtiny85-20SU-MCU_Microchip_ATtiny U1
 U 1 1 5B6F1978
 P 2200 2350
